File: dodgeball/dodgeball.kicad_sch (KiCad schematic)
At the start: 68 parts, among them J6 74HC04, J7 74HC74, J8 74LS10, J9 7402, K10 7402, K11 74LS04, M10 7400, P4 74HC00

Commit message: Updated Library Compatibility, Balls Fixed
New library is more parametrized to help with automatic converter: Delay and Video resistors. Balls now have appropriate fixes to keep them from sticking to walls.
Parts:
- removed CP28: 47, symbol Device:C_Small
- removed R47: 47000, symbol Device:R_Small
- removed R8: 220, symbol Device:R_US
- L9: C1_uF (none) -> 47; C2_uF (none) -> 10; R1_R (none) -> 47000; R2_R (none) -> 47000
Connections:
- net CREDIT LIGHT: now also K11.10
- net GND: now also F10.5 (I1a)
Other:
- moved on the sheet: D6A, E6A, F8B
