File: dodgeball/dodgeball_p2.kicad_sch (KiCad schematic)
At the start: 94 parts, among them J1 74LS20, J2 9316, J3 74LS10, J4 74LS107, J5 74LS20, J6 74HC04, J8 74LS10, K1 74LS93, K10 7402, K2 74LS04, K3 7400, K4 7400, K5 74LS04, K6 74LS93, K7 9316, K8 7400, M1 74LS93, M2 9316, M3 74LS10, M4 74LS74, M5 7402, M6 74LS74, M7 74LS93, M8 74LS93, P1 74LS93, P2 9316, P4 74HC00, P5 74LS93, P6 74LS107, P7 74LS93, P8 74LS93, Q5 2N3643, U9 LM741

Commit message: Updated Library Compatibility, Balls Fixed
New library is more parametrized to help with automatic converter: Delay and Video resistors. Balls now have appropriate fixes to keep them from sticking to walls.
Parts:
- removed C12: 10, symbol Device:C
- removed C13: 10u, symbol Device:C_Polarized_Small
- removed C13: 0.1u, symbol Device:C_Small
- removed C15: 1u, symbol Device:C_Polarized_Small
- removed Q5: 2N3643, Package_TO_SOT_THT:TO-92_Inline, symbol Transistor_BJT:2N3904
- removed R1: 47000, symbol Device:R
- removed R16, R17, R18, R49, R50, R51, R52, R53: 1000, symbol Device:R_US
- removed R20: 10K, symbol Device:R_US
- removed R21: 470k, symbol Device:R_US
- removed R22, R24: 100k, symbol Device:R_US
- removed R23: 1M, symbol Device:R_US
- removed U9: LM741, symbol Amplifier_Operational:LM741
- added U10, U11, U9: (no value), symbol DICE:DELAY
- added U8: (no value), symbol DICE:CLK_GATE
- L9: C1_uF (none) -> 47; C2_uF (none) -> 10; R1_R (none) -> 47000; R2_R (none) -> 47000
- U2: V1_R (none) -> 1000; V2_R (none) -> 1000; V3_R (none) -> 1000; V4_R (none) -> 1000; V5_R (none) -> 1000; V6_R (none) -> 1000; V7_R (none) -> 1000; V8_R (none) -> 1000000
Connections:
- net +5V: now also U2.1 (VIDEO1)
- net BALL VIDEO 1: now also U9.1 (I); no longer J4.9 (C)
- net BALL VIDEO 2: now also U10.1 (I); no longer J4.12 (C)
- net BALL VIDEO 3: now also U11.1 (I); no longer N4.9 (C)
- net CLOCK B: now also U8.3 (OUT); no longer K5.8
- net COMP SYNC: now also U2.2 (VIDEO2)
- net DEBRIS VIDEO: now also U2.7 (VIDEO7)
- net H GATE: now also U8.1 (IN)
- net OBJECT VIDEO 1: now also U2.5 (VIDEO5)
- net SCORE OUT: now also U2.3 (VIDEO3)
- net ~{OBJECT VIDEO 2}: now also U2.6 (VIDEO6)
- net ~{PLAY FIELD}: now also U2.4 (VIDEO4)
- net at N8.10: now also U4.Joystick::DOWN (Down); no longer U4.DOWN (down)
- net at K8.12: now also U4.Joystick::LEFT (Left); no longer U4.LEFT (left)
- net at K8.10, K8.13, K8.9: now also U4.Joystick::RIGHT (Right); no longer U4.RIGHT (right)
- net at N8.12, N8.13, N8.9: now also U4.Joystick::UP (Up); no longer U4.UP (up)
- net at N8.1, N8.4, N8.5: now also U3.Joystick::UP (Up); no longer U3.UP (up)
- net at N8.2: now also U3.Joystick::DOWN (Down); no longer U3.DOWN (down)
- net at K8.1: now also U3.Joystick::LEFT (Left); no longer U3.LEFT (left)
- net at K8.2, K8.4, K8.5: now also U3.Joystick::RIGHT (Right); no longer U3.RIGHT (right)
- new net: J4.12 (C), U10.2 (O)
- new net: K5.8, U8.2 (GATE)
- new net: N4.9 (C), U11.2 (O)
- new net: J4.9 (C), U9.2 (O)
Other:
- note added: "Note: Ball 4 finds itself nicely tucked where it wont bounce, this being a working solution to that issue."
